File: Hardware/ThunderBolt Nova - EAGLE CAD/ThunderBolt Nova Pico.sch (EAGLE design)
At the start: 32 parts, among them IC1 MCP73831/OT, U1 MCP1802T-3302I/OT

Commit message: corrections in examples
Parts:
- added U$3, U$4: PADSMD, 2brobots:PADSMD
- added U$8, U$9: FIDUCIAL, adafruit:FIDUCIAL
Connections:
- removed net N$10: C4.2, C5.2, C7.2, U1.GND
- net GND: now also C4.2, C5.2, C7.2, U$3.P$1, U1.GND
- net VBAT: now also U$4.P$1
Changed lines of the file:
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@@
 <part name="R7" library="adafruit" deviceset="R-US_" device="R0805" value="100k"/>
 <part name="C7" library="adafruit" deviceset="C-US" device="C0603K" value="0.1uF"/>
+<part name="U$3" library="2brobots" deviceset="PADSMD" device=""/>
+<part name="U$4" library="2brobots" deviceset="PADSMD" device=""/>
+<part name="U$8" library="adafruit" deviceset="FIDUCIAL" device=""/>
+<part name="U$9" library="adafruit" deviceset="FIDUCIAL" device=""/>
 </parts>
 <sheets>
@@
 <instance part="R7" gate="G$1" x="142.24" y="91.44" rot="R90"/>
 <instance part="C7" gate="G$1" x="68.58" y="58.42"/>
+<instance part="U$3" gate="G$1" x="132.08" y="5.08"/>
+<instance part="U$4" gate="G$1" x="129.54" y="17.78"/>
+<instance part="U$8" gate="G$1" x="7.62" y="5.08"/>
+<instance part="U$9" gate="G$1" x="15.24" y="5.08"/>
 </instances>
 <busses>
@@
 <pinref part="CN1" gate="G$1" pin="1"/>
 <wire x1="139.7" y1="12.7" x2="139.7" y2="7.62" width="0.1524" layer="91"/>
-<wire x1="139.7" y1="7.62" x2="119.38" y2="7.62" width="0.1524" layer="91"/>
+<wire x1="139.7" y1="7.62" x2="127" y2="7.62" width="0.1524" layer="91"/>
 <junction x="119.38" y="7.62"/>
+<pinref part="U$3" gate="G$1" pin="P$1"/>
+<wire x1="127" y1="7.62" x2="119.38" y2="7.62" width="0.1524" layer="91"/>
+<wire x1="127" y1="5.08" x2="127" y2="7.62" width="0.1524" layer="91"/>
+<junction x="127" y="7.62"/>
 </segment>
 <segment>
@@
 <junction x="215.9" y="66.04"/>
 <label x="208.28" y="66.04" size="1.778" layer="95"/>
+</segment>
+<segment>
+<pinref part="C5" gate="G$1" pin="2"/>
+<wire x1="78.74" y1="53.34" x2="78.74" y2="50.8" width="0.1524" layer="91"/>
+<pinref part="U1" gate="A" pin="GND"/>
+<wire x1="78.74" y1="50.8" x2="106.68" y2="50.8" width="0.1524" layer="91"/>
+<pinref part="C4" gate="G$1" pin="2"/>
+<wire x1="137.16" y1="55.88" x2="137.16" y2="40.64" width="0.1524" layer="91"/>
+<wire x1="137.16" y1="40.64" x2="106.68" y2="40.64" width="0.1524" layer="91"/>
+<wire x1="106.68" y1="40.64" x2="106.68" y2="50.8" width="0.1524" layer="91"/>
+<junction x="106.68" y="50.8"/>
+<pinref part="C7" gate="G$1" pin="2"/>
+<wire x1="68.58" y1="53.34" x2="68.58" y2="50.8" width="0.1524" layer="91"/>
+<wire x1="68.58" y1="50.8" x2="78.74" y2="50.8" width="0.1524" layer="91"/>
+<junction x="78.74" y="50.8"/>
+<label x="99.06" y="48.26" size="1.778" layer="95"/>
 </segment>
 </net>
@@
 </segment>
 </net>
-<net name="N$10" class="0">
-<segment>
-<pinref part="C5" gate="G$1" pin="2"/>
-<wire x1="78.74" y1="53.34" x2="78.74" y2="50.8" width="0.1524" layer="91"/>
-<pinref part="U1" gate="A" pin="GND"/>
-<wire x1="78.74" y1="50.8" x2="106.68" y2="50.8" width="0.1524" layer="91"/>
-<pinref part="C4" gate="G$1" pin="2"/>
-<wire x1="137.16" y1="55.88" x2="137.16" y2="40.64" width="0.1524" layer="91"/>
-<wire x1="137.16" y1="40.64" x2="106.68" y2="40.64" width="0.1524" layer="91"/>
-<wire x1="106.68" y1="40.64" x2="106.68" y2="50.8" width="0.1524" layer="91"/>
-<junction x="106.68" y="50.8"/>
-<pinref part="C7" gate="G$1" pin="2"/>
-<wire x1="68.58" y1="53.34" x2="68.58" y2="50.8" width="0.1524" layer="91"/>
-<wire x1="68.58" y1="50.8" x2="78.74" y2="50.8" width="0.1524" layer="91"/>
-<junction x="78.74" y="50.8"/>
-</segment>
-</net>
 <net name="VBAT" class="0">
 <segment>
@@
 <junction x="119.38" y="22.86"/>
 <pinref part="CN1" gate="G$1" pin="2"/>
-<wire x1="119.38" y1="22.86" x2="139.7" y2="22.86" width="0.1524" layer="91"/>
+<wire x1="119.38" y1="22.86" x2="124.46" y2="22.86" width="0.1524" layer="91"/>
+<wire x1="124.46" y1="22.86" x2="139.7" y2="22.86" width="0.1524" layer="91"/>
 <wire x1="139.7" y1="22.86" x2="139.7" y2="15.24" width="0.1524" layer="91"/>
-</segment>
-<segment>
+<pinref part="U$4" gate="G$1" pin="P$1"/>
+<wire x1="124.46" y1="17.78" x2="124.46" y2="22.86" width="0.1524" layer="91"/>
+<junction x="124.46" y="22.86"/>
+</segment>
+<segment>
